Commit message: Gazebo sim done, moves with teleop twist keyboard. URDF data given to Gazebo diff_drive controller, which takaes /cmd_vel input and returns joint_states as output to the publisher

File: description/robot.urdf.xacro (robot description, xacro)
@@ -2,3 +2,4 @@
 <robot xmlns:xacro="http://www.ros.org/wiki/xacro"  name="robot">
     <xacro:include filename="robot_core.xacro"/>
+    <xacro:include filename="gazebo_control.xacro"/>
 </robot>

File: description/robot_core.xacro (robot description, xacro)
@@ -19,4 +19,5 @@
     <link name="base_link">
     </link>
+    <!-- CHASSIS -->
     <joint name="chassis_joint" type="fixed">
         <parent link="base_link"/>
@@ -42,4 +43,8 @@
         </xacro:inertial_box>
     </link>
+    <gazebo reference="chassis">
+        <material>Gazebo/Orange</material>
+    </gazebo>
+    <!-- LEFT_WHEEL -->
     <joint name="left_wheel_joint" type="continuous">
         <parent link="base_link"/>
@@ -64,4 +69,8 @@
         </xacro:inertial_cylinder>
     </link>
+    <gazebo reference="left_wheel">
+        <material>Gazebo/Blue</material>
+    </gazebo>
+    <!-- RIGHT_WHEEL -->
     <joint name="right_wheel_joint" type="continuous">
         <parent link="base_link"/>
@@ -86,4 +95,8 @@
         </xacro:inertial_cylinder>
     </link>
+    <gazebo reference="right_wheel">
+        <material>Gazebo/Blue</material>
+    </gazebo>
+    <!-- CASTOR_WHEEL -->
     <joint name="castor_wheel_joint" type="fixed">
         <parent link="chassis"/>
@@ -107,3 +120,8 @@
         </xacro:inertial_sphere>
     </link>
+    <gazebo reference="castor_wheel">
+        <material>Gazebo/Blue</material>
+        <mu1 value="0.001"/>
+        <mu2 value="0.002"/>
+    </gazebo>
 </robot>
